Commit message: Fix URDF physics: odom scale, caster height, wheel contact
- DiffDrive: use wheel_radius (gz-sim ignores wheel_diameter and fell
  back to its 0.2 m default, so the robot drove at 1/4 of the commanded
  speed while /odom reported the full speed); drop params gz-sim does
  not recognize and use max_linear_acceleration instead.
- Lower casters so their bottoms are level with the drive wheels
  (they floated 3.5 cm above ground, the chassis pitched ~14 deg).
- Give casters zero friction so they don't drag.
- Use sphere collisions for the wheels: cylinder contacts landed on the
  inner wheel edges (effective track 0.27 m vs 0.30 m), so in-place turns
  were under-reported by ~10% in /odom.
- Correct inertia (chassis COM at its center, box/cylinder formulas),
  remove IMU collision, use exact 1-degree lidar beam spacing.

Verified in Gazebo: straight-line and turning odom match ground truth
within 0.3%; slam_toolbox map has 0 ghost cells, SLAM pose error 0.9 cm
mean over a full loop.

Co-Authored-By: Claude Opus 5.5 <noreply@anthropic.com>

File: diff_robot_description/urdf/diff_robot.urdf.xacro (robot description, xacro)
@@ -11,8 +11,6 @@
   <!-- ============================================================= -->
 <robot xmlns:xacro="http://www.ros.org/wiki/xacro" name="diff_robot">
-  <xacro:property name="base_width"   value="0.30" />   <!-- 轮距 L (m)
--->
-  <xacro:property name="wheel_radius" value="0.05" />   <!-- 轮半径 r (m)
--->
+  <xacro:property name="base_width"   value="0.30" />   <!-- 轮距 L (m)                   -->
+  <xacro:property name="wheel_radius" value="0.05" />   <!-- 轮半径 r (m)                 -->
   <xacro:property name="base_length"  value="0.25" />   <!-- 底盘长 (m)                    -->
   <xacro:property name="base_height"  value="0.08" />   <!-- 底盘高 (m)                    -->
@@ -53,8 +51,10 @@
   </collision>
   <inertial>
+    <!-- 质心在底盘几何中心，惯量按均匀长方体公式 m(a²+b²)/12 计算 -->
+    <origin xyz="0 0 ${base_height/2}" rpy="0 0 0"/>
     <mass value="1.0"/>
-    <inertia ixx="0.01" ixy="0.0" ixz="0.0"
-             iyy="0.01" iyz="0.0"
-             izz="0.02"/>
+    <inertia ixx="${(base_width*base_width + base_height*base_height)/12}" ixy="0.0" ixz="0.0"
+             iyy="${(base_length*base_length + base_height*base_height)/12}" iyz="0.0"
+             izz="${(base_length*base_length + base_width*base_width)/12}"/>
   </inertial>
 </link>
@@ -71,15 +71,19 @@
       <material name="wheel_color"/>
     </visual>
+    <!-- collision 用球体而不是圆柱：圆柱和地面的接触点会落在轮子内侧边缘
+         （y=±0.135），实际转向轮距变成 0.27m，而 DiffDrive 按 0.30m 算 odom，
+         实测原地转向 odom 少报约 10%。球体接触点正好在轮子中线上，
+         实测 odom 与真值一致。visual 仍是圆柱，外观不变。 -->
     <collision>
       <geometry>
-        <cylinder radius="${wheel_radius}" length="${wheel_width}"/>
-      </geometry>
-      <origin xyz="0 0 0" rpy="${pi/2} 0 0"/>
+        <sphere radius="${wheel_radius}"/>
+      </geometry>
     </collision>
     <inertial>
+      <!-- 均匀圆柱体：转轴(Y) = mr²/2，其余 = m(3r²+h²)/12 -->
       <mass value="0.05"/>
-      <inertia ixx="0.0001" ixy="0.0" ixz="0.0"
-               iyy="0.0001" iyz="0.0"
-               izz="0.0001"/>
+      <inertia ixx="${0.05*(3*wheel_radius*wheel_radius + wheel_width*wheel_width)/12}" ixy="0.0" ixz="0.0"
+               iyy="${0.05*wheel_radius*wheel_radius/2}" iyz="0.0"
+               izz="${0.05*(3*wheel_radius*wheel_radius + wheel_width*wheel_width)/12}"/>
     </inertial>
   </link>
@@ -92,5 +96,5 @@
   <!-- 左轮关节: 连续旋转 (continuous)，绕 Y 轴旋转                   -->
   <!-- 位置: 底盘左侧 (x=0, y=+base_width/2, z=-wheel_radius)       -->
-  <!--        z 向下偏移使得车轮底部刚好接触地面                     -->
+  <!--        车轮顶部贴着底盘底面，车轮底部在 base_link 下方 2r 处（即地面） -->
   <joint name="left_wheel_joint" type="continuous">
     <parent link="base_link"/>
@@ -111,15 +115,16 @@
       <material name="wheel_color"/>
     </visual>
+    <!-- 同左轮：collision 用球体，接触点在轮子中线上 -->
     <collision>
       <geometry>
-        <cylinder radius="${wheel_radius}" length="${wheel_width}"/>
-      </geometry>
-      <origin xyz="0 0 0" rpy="${pi/2} 0 0"/>
+        <sphere radius="${wheel_radius}"/>
+      </geometry>
     </collision>
     <inertial>
+      <!-- 均匀圆柱体：转轴(Y) = mr²/2，其余 = m(3r²+h²)/12 -->
       <mass value="0.05"/>
-      <inertia ixx="0.0001" ixy="0.0" ixz="0.0"
-               iyy="0.0001" iyz="0.0"
-               izz="0.0001"/>
+      <inertia ixx="${0.05*(3*wheel_radius*wheel_radius + wheel_width*wheel_width)/12}" ixy="0.0" ixz="0.0"
+               iyy="${0.05*wheel_radius*wheel_radius/2}" iyz="0.0"
+               izz="${0.05*(3*wheel_radius*wheel_radius + wheel_width*wheel_width)/12}"/>
     </inertial>
   </link>
@@ -166,5 +171,6 @@
     <parent link="base_link"/>
     <child link="front_caster_link"/>
-    <origin xyz="${base_length/2 + 0.02} 0 ${-wheel_radius}" rpy="0 0 0"/>
+    <!-- 万向轮底部与驱动轮底部齐平（都在 z = -2r），否则会悬空导致车身前后倾斜 -->
+    <origin xyz="${base_length/2 + 0.02} 0 ${-(2*wheel_radius - caster_radius)}" rpy="0 0 0"/>
   </joint>
   <link name="rear_caster_link">
@@ -192,6 +198,15 @@
     <parent link="base_link"/>
     <child link="rear_caster_link"/>
-    <origin xyz="${-base_length/2 - 0.02} 0 ${-wheel_radius}" rpy="0 0 0"/>
-  </joint>
+    <origin xyz="${-base_length/2 - 0.02} 0 ${-(2*wheel_radius - caster_radius)}" rpy="0 0 0"/>
+  </joint>
+  <!-- 万向轮零摩擦：固定关节的球体不会滚动，有摩擦就会拖地、转弯时干扰里程计 -->
+<gazebo reference="front_caster_link">
+  <mu1>0.0</mu1>
+  <mu2>0.0</mu2>
+</gazebo>
+<gazebo reference="rear_caster_link">
+  <mu1>0.0</mu1>
+  <mu2>0.0</mu2>
+</gazebo>
   <!-- ============================================================= -->
   <!-- 7. 激光雷达 (laser_link) - 安装在底盘顶部                    -->
@@ -248,10 +263,5 @@
       <material name="sensor_color"/>
     </visual>
-    <collision>
-      <geometry>
-        <box size="0.03 0.03 0.02"/>
-      </geometry>
-      <origin xyz="0 0 0" rpy="0 0 0"/>
-    </collision>
+    <!-- 不设 collision：IMU 在底盘内部，碰撞由底盘 collision box 承担 -->
     <inertial>
       <mass value="0.01"/>
@@ -287,7 +297,11 @@
     <right_joint>right_wheel_joint</right_joint>
     <wheel_separation>${base_width}</wheel_separation>
-    <wheel_diameter>${2 * wheel_radius}</wheel_diameter>
-    <max_wheel_torque>50</max_wheel_torque>
-    <max_wheel_acceleration>5.0</max_wheel_acceleration>
+    <!-- 注意：gz-sim DiffDrive 只认 wheel_radius，不认 wheel_diameter。
+         写成 wheel_diameter 会被静默忽略、退回默认半径 0.2m（实际 0.05m），
+         导致实际速度只有指令的 1/4，而 /odom 却按指令速度报告。
+         max_wheel_torque / max_wheel_acceleration 也是老插件的参数名，
+         gz-sim 里对应的是 max_linear_acceleration / max_angular_acceleration。 -->
+    <wheel_radius>${wheel_radius}</wheel_radius>
+    <max_linear_acceleration>${5.0 * wheel_radius}</max_linear_acceleration>
     <topic>cmd_vel</topic>
     <odom_topic>odom</odom_topic>
@@ -306,6 +320,4 @@
     <frame_id>odom</frame_id>
     <child_frame_id>base_link</child_frame_id>
-    <publish_odom>true</publish_odom>
-    <publish_odom_tf>true</publish_odom_tf>
   </plugin>
 </gazebo>
@@ -343,6 +355,7 @@
          <samples>360</samples>
          <resolution>1</resolution>
-         <min_angle>-3.14</min_angle>
-        <max_angle>3.14</max_angle>
+         <!-- 360 束、每束 1°：首尾不重叠，最后一束在 π - 1° -->
+         <min_angle>${-pi}</min_angle>
+         <max_angle>${pi - 2*pi/360}</max_angle>
        </horizontal>
        <vertical>
